File: mainboard/3.3V_Analog.kicad_sch (KiCad schematic)
At the start: 9 parts, among them U18 TPS7A4701RGWR

Commit message: Initial layout completed
Parts:
- U18: footprint TPS7A4701RGWR_new:RGW0020A-MFG -> TPS7A:RGW0020A-IPC_A
Changed lines of the file:
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@@
 			)
 		)
-		(property "Footprint" "TPS7A4701RGWR_new:RGW0020A-MFG"
+		(property "Footprint" "TPS7A:RGW0020A-IPC_A"
 			(at 119.38 76.2 0)
 			(hide yes)
