File: mainboard/mainboard.kicad_pcb (KiCad board)
At the start: 6 copper layers, 60 x 48 mm, 235 parts, among them J6 Conn_01x08_Pin, J7 ARM/JTAG, J8 Conn_01x02_Pin, U1 DRV8323SRTAR, U10 CSD88599Q5DC, U11 CSD88599Q5DC, U12 CSD88599Q5DC, U13 CSD88599Q5DC, U14 CSD88599Q5DC, U15 CSD88599Q5DC, U16 CSD88599Q5DC, U17 TPS54360BDDAR, U18 TPS7A4701RGWR, U2 DRV8323SRTAR, U3 DRV8323SRTAR, U4 DRV8323SRTAR, U5 CSD88599Q5DC, U6 CSD88599Q5DC, U7 CSD88599Q5DC, U8 CSD88599Q5DC, U9 CSD88599Q5DC

Commit message: First proto hardware
Parts:
- added C100: 1nF, Capacitor_SMD:C_0201_0603Metric, F.Cu at (92.4, 90.0)
- added C89: 1nF, Capacitor_SMD:C_0201_0603Metric, F.Cu at (111.5, 114.7)
- added C90: 1nF, Capacitor_SMD:C_0201_0603Metric, F.Cu at (111.2, 113.4)
- added C91: 1nF, Capacitor_SMD:C_0201_0603Metric, F.Cu at (107.5, 108.4)
- added C92: 1nF, Capacitor_SMD:C_0201_0603Metric, F.Cu at (110.8, 93.0)
- added C93: 1nF, Capacitor_SMD:C_0201_0603Metric, F.Cu at (110.9, 90.8)
- added C94: 1nF, Capacitor_SMD:C_0201_0603Metric, F.Cu at (107.3, 87.2)
- added C95: 1nF, Capacitor_SMD:C_0201_0603Metric, F.Cu at (88.9, 106.8)
- added C96: 1nF, Capacitor_SMD:C_0201_0603Metric, F.Cu at (89.4, 109.3)
- added C97: 1nF, Capacitor_SMD:C_0201_0603Metric, F.Cu at (91.8, 113.0)
- added C98: 1nF, Capacitor_SMD:C_0201_0603Metric, F.Cu at (88.8, 84.5)
- added C99: 1nF, Capacitor_SMD:C_0201_0603Metric, F.Cu at (88.7, 85.8)
- C29, C33, C37, C41, C45, C49, C53, C57, C61, C65, C69, C73: value 2.2uF -> 10uF
- D1: moved to B.Cu
Routing:
- net M2_SNB: track 11.1 -> 11.8 mm
- net M3_BEMFC: track 48.6 -> 48.0 mm
- net M1_SNA: track 15.9 -> 16.5 mm
- net M3_SPB: track 12.6 -> 13.1 mm
- net nFAULTM4: vias 3 -> 2
- net VBAT_SNS: vias 1 -> 0
- net M3_LSB: vias 8 -> 7
- net M2_IC: vias 2 -> 1
- net M2_IA: vias 2 -> 1
- net M1_PWMC: vias 2 -> 1
- net M1_PWMB: vias 2 -> 1
- net M1_PWMA: vias 2 -> 1
Other:
- board text added: "+"
- board text added: "-"
- board text added: "-GND-"
- board text added: "1"
- board text added: "2"
- board text added: "3"
- board text added: "3V3"
- board text added: "4"
- board text added: "A"
- board text added: "B"
- board text added: "BeagleConnect Quad ESC BeagleBoard.org"
- board text added: "C"
- board text added: "EN"
- board text added: "REV A2"
- board text added: "SWCLK"
- board text added: "SWDIO"
- board text added: "SWO"
- board text added: "T"
- board text added: "TDI"
- board text added: "nRST"
