File: mainboard/interface.kicad_sch (KiCad schematic)
At the start: 19 parts, among them J10 MikroBUS R, J6 Conn_01x08_Pin, J7 ARM/JTAG, J8 MikroBUS L

Commit message: Initial layout completed
Parts:
- removed J10: MikroBUS R, symbol Connector:Conn_01x12_Socket
- removed J8: MikroBUS L, symbol Connector:Conn_01x12_Socket
- removed R13, R14, R15, R16, R17: 0, Resistor_SMD:R_0402_1005Metric, symbol RC0603FR-0710KL:RC0603FR-0710KL
- added J8: Conn_01x02_Pin, Connector_PinHeader_1.00mm:PinHeader_1x02_P1.00mm_Vertical, symbol Connector:Conn_01x02_Pin
- J7: footprint (none) -> Connector_PinHeader_1.27mm:PinHeader_2x05_P1.27mm_Vertical_SMD; now fitted
- J9: footprint LGA100_1.0mm_0.5x0.3NSMD_SoM:LGA-100_10x10_14.0x14.0mm -> AM13E_SoM_Receptacle_LGA100:AM13E_SoM_Receptacle_LGA100
Connections:
- net BSL_INVOKE is gone; now on net nFAULTM1: J9.K2
- net CAN_RX is gone; now on net DSHOT2: J9.A1
- net CAN_TX is gone; now on net M4_IC: J9.A2
- net DSHOT1_IO is gone; now on net DSHOT1: J6.5 (Pin_5)
- net DSHOT2_IO is gone; now on net DSHOT2: J6.6 (Pin_6)
- net DSHOT3_IO is gone; now on net DSHOT3: J6.7 (Pin_7)
- net DSHOT4_IO is gone; now on net DSHOT4: J6.8 (Pin_8)
- net FC_Telemetry_IO is gone; now on net FC_Telemetry: J6.4 (Pin_4)
- net +3.3V: now also J9.5
- net DRV_ENABLE: now also J9.G8; no longer J9.K4
- net DSHOT1: now also J9.H3; no longer J9.A7
- net DSHOT2: no longer J9.A6
- net DSHOT3: now also J9.J4; no longer J9.A5
- net DSHOT4: now also J9.J1; no longer J9.A4
- net FC_Current: now also J9.H9; no longer J9.A9
- net FC_Telemetry: now also J9.F8; no longer J9.A10
- net GND: now also J9.1, J9.2, J9.3, J9.4, J9.D4, J9.D6, J9.E5, J9.E7, J9.F4, J9.F6, J9.G5, J9.G7, J8.1 (Pin_1)
- net INL_ENABLE: now also J9.H10; no longer J9.A8
- net M1_BEMFA: now also J9.H2; no longer J9.B4
- net M1_BEMFB: now also J9.F2; no longer J9.B3
- net M1_BEMFC: now also J9.F3; no longer J9.B2
- net M1_IA: now also J9.H1; no longer J9.B7
- net M1_IB: now also J9.G1; no longer J9.B6
- net M1_IC: now also J9.J2; no longer J9.B5
- net M1_PWMA: now also J9.H6; no longer J9.B10
- net M1_PWMB: now also J9.K6; no longer J9.B9
- net M1_PWMC: now also J9.J6; no longer J9.B8
- net M2_BEMFA: now also J9.E3; no longer J9.D4
- net M2_BEMFB: now also J9.D2; no longer J9.D3
- net M2_BEMFC: now also J9.C2; no longer J9.D2
- net M2_IA: now also J9.C1; no longer J9.D7
- net M2_IB: now also J9.D1; no longer J9.D6
- net M2_IC: now also J9.D3; no longer J9.D5
- net M2_PWMA: now also J9.A6; no longer J9.D10
- net M2_PWMB: now also J9.B6; no longer J9.D9
- net M2_PWMC: now also J9.B4; no longer J9.D8
- net M3_BEMFA: now also J9.K4; no longer J9.F4
- net M3_BEMFB: now also J9.B5; no longer J9.F3
- net M3_BEMFC: now also J9.H5; no longer J9.F2
- net M3_IA: now also J9.K3; no longer J9.F7
- net M3_IB: now also J9.K5; no longer J9.F6
- net M3_IC: now also J9.H4; no longer J9.F5
- net M3_PWMA: now also J9.A7; no longer J9.F10
- net M3_PWMB: now also J9.J8; no longer J9.F9
- net M3_PWMC: now also J9.B10; no longer J9.F8
- net M4_BEMFA: now also J9.A4; no longer J9.H4
- net M4_BEMFB: now also J9.K8; no longer J9.H3
- net M4_BEMFC: now also J9.E2; no longer J9.H2
- net M4_IA: now also J9.B3; no longer J9.H7
- net M4_IB: now also J9.J7; no longer J9.H6
- net M4_IC: no longer J9.H5
- net M4_PWMA: now also J9.A10; no longer J9.H10
- net M4_PWMB: now also J9.A9; no longer J9.H9
- net M4_PWMC: now also J9.C9; no longer J9.H8
- net M_TEMP1: now also J9.F1; no longer J9.B1
- net M_TEMP2: now also J9.B2; no longer J9.D1
- net M_TEMP3: now also J9.G3; no longer J9.F1
- net M_TEMP4: now also J9.E1; no longer J9.H1
- net SPI_MISO: now also J9.B8; no longer J9.K6
- net SPI_MOSI: now also J9.C7; no longer J9.K5
- net SPI_SCLK: now also J9.C8; no longer J9.K7
- net SPI_nCSM1: now also J9.G2; no longer J9.C9
- net SPI_nCSM2: now also J9.B7; no longer J9.E9
- net SPI_nCSM3: now also J9.H7; no longer J9.G9
- net SPI_nCSM4: now also J9.A8; no longer J9.J9
- net SWCLK: now also J9.J9; no longer J9.K9
- net SWO: now also J9.E9; no longer J9.K8
- net TDI: now also J9.J10; no longer J9.J1
- net VAA: now also J9.F5; no longer J9.K1
- net VBAT_SNS: now also J9.J5; no longer J9.K3
- net nFAULTM1: no longer J9.C10
- net nFAULTM2: now also J9.C6; no longer J9.E10
- net nFAULTM4: now also J9.A5; no longer J9.J10
- net nRST: now reaches J9.C5
- net nRST: now also J7.10 (Pin_10)
- net +5V: now reaches J9.E4
- net +5V: now also J9.D5, J9.D7, J9.E6, J9.F7, J9.G4, J9.G6
- net NRST: no longer names the net of J9.A3
- net NRST: no longer J7.10 (Pin_10)
- new net BUZZER: J8.2 (Pin_2), J9.F9
- no-connect marks 22 -> 19

Commit message: Use BeagleConnect product names consistently
Other:
- title: AM13E QuadESC Mainboard — Interface -> BeagleConnect QuadESC Mainboard — Interface
Changed lines of the file:
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@@
 	(paper "USLetter")
 	(title_block
-		(title "AM13E QuadESC Mainboard — Interface")
+		(title "BeagleConnect QuadESC Mainboard — Interface")
 		(date "2026-08-06")
 		(rev "A")
