File: mainboard/power.kicad_sch (KiCad schematic)
At the start: 3 parts

Commit message: Use BeagleConnect product names consistently
Other:
- title: AM13E QuadESC Mainboard — Power -> BeagleConnect QuadESC Mainboard — Power
Changed lines of the file:
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@@
 	(paper "USLetter")
 	(title_block
-		(title "AM13E QuadESC Mainboard — Power")
+		(title "BeagleConnect QuadESC Mainboard — Power")
 		(date "2026-08-06")
 		(rev "A")
