File: som/som.kicad_pcb (KiCad board)
At the start: 4 copper layers, 25.4 x 38.1 mm, 58 parts, among them J2 ZEPTO_DEBUG, J3 MikroBUS L, J4 Qwiic, J5 Drone_CAN, J6 MikroBUS R, U1 XAM13E23019GTPZ, U2 TCAN844DRBRQ1, U3 TS5A3166YZPR, U4 TPS2116DRLR, U5 TPS22950YBHR, U6 TPS7A2633DRVR, Y1 ECS-250-12-33-AGN-TR

Commit message: First proto hardware
Parts:
- added G***: LOGO, Upside Down Labs (Graphics):mikroBUS-12mm, B.Cu at (100.2, 106.3)
- added R21: 10k, Resistor_SMD:R_0201_0603Metric, F.Cu at (102.6, 89.3)
- added kibuzzard-698ADC75: G***, kibuzzard-698ADC75, B.Cu at (93.6, 115.0)
- added kibuzzard-698ADC7E: G***, kibuzzard-698ADC7E, B.Cu at (96.1, 114.9)
- added kibuzzard-698ADC83: G***, kibuzzard-698ADC83, B.Cu at (98.7, 114.8)
- added kibuzzard-698ADC88: G***, kibuzzard-698ADC88, B.Cu at (101.2, 114.9)
- added kibuzzard-698ADC8D: G***, kibuzzard-698ADC8D, B.Cu at (103.7, 114.9)
- added kibuzzard-698ADC92: G***, kibuzzard-698ADC92, B.Cu at (106.3, 115.0)
- added kibuzzard-698ADC96: G***, kibuzzard-698ADC96, B.Cu at (108.8, 114.9)
- added kibuzzard-698AE4C9: G***, kibuzzard-698AE4C9, B.Cu at (91.0, 115.0)
- added kibuzzard-698CA76F: G***, kibuzzard-698CA76F, B.Cu at (100.0, 91.0)
Connections:
- J3 pad 1: unconnected-(J3-Pin_1-Pad1) -> GND
- J3 pad 2: unconnected-(J3-Pin_2-Pad2) -> PA19
- J3 pad 3: unconnected-(J3-Pin_3-Pad3) -> PA15
- J3 pad 4: unconnected-(J3-Pin_4-Pad4) -> VAA
- J6 pad 1: unconnected-(J6-Pin_1-Pad1) -> GND
- J6 pad 2: unconnected-(J6-Pin_2-Pad2) -> CANL
- J6 pad 3: unconnected-(J6-Pin_3-Pad3) -> CANH
- J6 pad 4: unconnected-(J6-Pin_4-Pad4) -> +5V
Routing:
- net PA15: track 2.21 -> 31.1 mm
- net PA19: track 3.53 -> 27.8 mm
- net VAA: track 14.9 -> 26.5 mm
- net CANH: track 10.4 -> 17.3 mm, vias 0 -> 1
- net +3.3V: track 125.0 -> 130.0 mm, vias 8 -> 9
- net CANL: track 15.7 -> 20.6 mm
- net CAN_TERM: track 38.3 -> 41.7 mm
- net +5V: track 84.8 -> 86.0 mm
- net GND: track 50.0 -> 49.0 mm
Other:
- board text added: "3V3"
- board text added: "5V"
- board text added: "AN"
- board text added: "BRX"
- board text added: "BSL"
- board text added: "BTX"
- board text added: "BeagleBoard.org"
- board text added: "BeagleConnect"
- board text added: "CANH"
- board text added: "CANL"
- board text added: "CH"
- board text added: "CIPO"
- board text added: "CL"
- board text added: "CLK"
- board text added: "COPI"
- board text added: "CS"
- board text added: "DIO"
- board text added: "GND"
- board text added: "INT"
- board text added: "PWM"
- board text added: "PWR"
- board text added: "RST"
- board text added: "RX"
- board text added: "SCK"
- board text added: "SCL"
- board text added: "SDA"
- board text added: "STAT"
- board text added: "SWO"
- board text added: "TDI"
- board text added: "TX"
- board text added: "VAA"
