File: som/can-transceiver.kicad_sch (KiCad schematic)
At the start: 13 parts, among them U2 TCAN844DRBRQ1

Commit message: Initial layout completed
Parts:
- removed C17: 4.7nF, Capacitor_SMD:C_0201_0603Metric, symbol GRM1555C1H472JE01D:GRM1555C1H472JE01D
- removed R16, R19: 60.4, Resistor_SMD:R_0201_0603Metric, symbol Device:R
- removed R17, R18: 0, Resistor_SMD:R_0201_0603Metric, symbol Device:R
- added R10: 120, Resistor_SMD:R_1206_3216Metric, symbol Device:R
- added U3: TS5A3166YZPR, TS5A3166:YZP5, symbol TS5A3166:TS5A3166YZPR
- renumbered C14 to C15, C15 to C16, C16 to C17, R14 to R8, R15 to R9
Connections:
- net +5V: now also U3.A2
- net CANH: now also L1.4, R10.1; no longer L1.3
- net CANL: now also L1.3, U3.B1; no longer L1.4
- net GND: now also U3.C1
- net at R9.2, U2.6 (CANL): now also L1.2; no longer L1.1
- net at R8.1, U2.7 (CANH): now also L1.1; no longer L1.2
- net +3V3 renamed +3.3V
- new net CAN_TERM: U3.C2
- new net SW_NO: R10.2, U3.A1

Commit message: First proto hardware
Changed lines of the file:
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@@
 		(in_pos_files yes)
 		(dnp no)
-		(fields_autoplaced yes)
 		(property "Reference" "U3"
 			(at 173.99 130.81 0)
@@
 		)
 		(property "Value" "TS5A3166YZPR"
-			(at 173.99 133.35 0)
+			(at 173.736 133.858 0)
 			(show_name no)
 			(do_not_autoplace no)

Commit message: Use BeagleConnect product names consistently
Other:
- title: AM13E QuadESC SoM — CAN transceiver -> BeagleConnect Torque — CAN transceiver
Changed lines of the file:
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@@
 	(paper "USLetter")
 	(title_block
-		(title "AM13E QuadESC SoM — CAN transceiver")
+		(title "BeagleConnect Torque — CAN transceiver")
 		(date "2026-08-06")
 		(rev "A")
