File: som/io-connectors.kicad_sch (KiCad schematic)
At the start: 6 parts, among them J1 Qwiic, J2 Drone_CAN, J3 ZEPTO_DEBUG, J5 MikroBUS L, J6 MikroBUS R

Commit message: Initial layout completed
Parts:
- added D1, D2: LED, LED_SMD:LED_0402_1005Metric, symbol Device:LED
- added R11, R12: 2.2k, Resistor_SMD:R_0201_0603Metric, symbol RC0603FR-07100KL:RC0603FR-07100KL
- added R13: 1.5k, Resistor_SMD:R_0201_0603Metric, symbol RC0603FR-07100KL:RC0603FR-07100KL
- added R14, R17: 10k, Resistor_SMD:R_0201_0603Metric, symbol RC0603FR-07100KL:RC0603FR-07100KL
- added R15, R16: 4.7k, Resistor_SMD:R_0201_0603Metric, symbol RC0603FR-07100KL:RC0603FR-07100KL
- J1: renamed from J4; now fitted
- renumbered J3 to J2, J5 to J3, J1 to J4, J2 to J5
Connections:
- net DSHOT1 is gone; now on net CAN_RX: J1.K9
- net M1_BEMFC is gone; now on net BSL_INVOKE: J1.B1
- net M2_IA is gone; now on net GND: J1.D6
- net M2_IB is gone; now on net +VDC: J1.D5
- net M2_IC is gone; now on net GND: J1.D4
- net M2_PWMA is gone; now on net BSL_I2C_SDA: J1.D9
- net M2_PWMC is gone; now on net +VDC: J1.D7
- net M3_IA is gone; now on net GND: J1.F6
- net M3_IC is gone; now on net GND: J1.F4
- net M3_PWMC is gone; now on net +VDC: J1.F7
- net M4_PWMB is gone; now on net CAN_TX: J1.H8
- net M_TEMP1 is gone; now on net BSL_I2C_SCL: J1.C10
- net PWM is gone; now on net PB12: J3.5 (Pin_5)
- net RST is gone; now on net PA20: J6.6 (Pin_6)
- net SPI_nCS2 is gone; now on net PA21: J1.D10
- net UART_RX is gone; now on net PB22: J3.8 (Pin_8)
- net UART_TX is gone; now on net PB21: J3.7 (Pin_7)
- net VBAT_SNS is gone; now on net PA13: J1.K10
- net VREF_IN is gone; now on net AN: J1.K1
- net nFAULT4 is gone; now on net PA14: J1.J9
- net +3.3V: now also R11.1, R12.1, R13.1, R14.1, R15.1, R16.1
- net BSL_I2C_SCL: now also R16.2
- net BSL_I2C_SDA: now also R15.2
- net BSL_INVOKE: now also R17.2; no longer J1.K2
- net BSL_UART_RX: now also J1.C3
- net BSL_UART_TX: now also J1.A3
- net CAN_RX: no longer J1.A8
- net CAN_TX: no longer J1.A9
- net GND: now also J1.E5, J1.E7, J1.G5, J1.G7, D2.1 (K), R17.1
- net INT: now also J1.C4
- net PA16: now reaches J1.C1
- net PB5: now reaches J1.C2
- net nRST: now reaches J1.C5
- net nRST: now also J2.7 (Pin_7)
- net PB15: now reaches J1.C6
- net PC6: now reaches J1.C7
- net PC6: now also J6.10 (Pin_10)
- net PC2: now reaches J1.C8
- net PC2: now also J6.8 (Pin_8)
- net PC8: now reaches J1.E1
- net PC7: now reaches J1.E2
- net PA17: now reaches J1.E3
- net +VDC: now reaches J1.E4
- net +VDC: now also J1.E6, J1.G4, J1.G6
- net PB22: now reaches J1.E8
- net PC12: now reaches J1.G1
- net PC13: now reaches J1.G2
- net PB25: now reaches J1.G3
- net PB10: now reaches J1.G8
- net PA29: now reaches J1.J2
- net PA31: now reaches J1.J3
- net PB28: now reaches J1.J4
- net PB31: now reaches J1.J5
- net PB8: now reaches J1.J6
- net PA8: now reaches J1.J7
- net PA10: now reaches J1.J8
- net DRV_ENABLE renamed PC1
- net DSHOT2 renamed PA9
- net DSHOT3 renamed PB9
- net DSHOT4 renamed PB7
- net FC_Current renamed PB24
- net FC_Telemetry renamed PB27
- net INL_ENABLE renamed PB30
- net M1_BEMFA renamed PA3
- net M1_BEMFB renamed PA5
- net M1_IA renamed PC26
- net M1_IB renamed PB1
- net M1_IC renamed PC18
- net M1_PWMA renamed CAN_TERM
- net M1_PWMB renamed PC4
- net PC4: now also J6.9 (Pin_9), R13.2
- net M1_PWMC renamed PB14
- net M2_BEMFA renamed PA7
- net M2_BEMFB renamed PB4
- net M2_BEMFC renamed PA18
- net M2_PWMB renamed PA20
- net M3_BEMFA renamed PC9
- net M3_BEMFB renamed PC11
- net M3_BEMFC renamed PC10
- net M3_IB renamed VAA
- net M3_PWMA renamed PB19
- net M3_PWMB renamed PB21
- net M4_BEMFA renamed PC15
- net M4_BEMFB renamed PC14
- net M4_BEMFC renamed PA27
- net M4_IA renamed PB6
- net M4_IB renamed PB29
- net M4_IC renamed PB26
- net M4_PWMA renamed PB12
- net M4_PWMC renamed PB16
- net M_TEMP2 renamed PB23
- net M_TEMP3 renamed PB17
- net M_TEMP4 renamed PA15
- net NRST renamed PA4
- net PA4: no longer J2.7 (Pin_7)
- net SPI_CS_MB renamed PA21
- net PA21: now also R14.2
- net SPI_MISO renamed PB0
- net PB0: no longer J6.9 (Pin_9)
- net SPI_MOSI renamed PB13
- net PB13: no longer J6.10 (Pin_10)
- net SPI_SCLK renamed PC25
- net PC25: no longer J6.8 (Pin_8)
- net SPI_nCS1 renamed PA25
- net SPI_nCS3 renamed PB20
- net SPI_nCS4 renamed PB11
- net SWCLK renamed PA14
- net PA14: no longer J1.A3
- net SWDIO renamed PA13
- net PA13: no longer J1.A4
- net SWO renamed PA2
- net TDI renamed PA26
- net nFAULT1 renamed PA24
- net nFAULT2 renamed PA19
- net nFAULT3 renamed PB18
- net PB18: now also D1.1 (K)
- new net: D1.2 (A), R12.2
- new net: D2.2 (A), R11.2
- new net PA30: J1.K2
- new net PB3: J1.A4
- new net PC3: J1.A9
- new net PC5: J1.A8
Other:
- moved on the sheet: J2, J3, J4, J5, J6

Commit message: First proto hardware
Parts:
- added R21: 10k, Resistor_SMD:R_0201_0603Metric, symbol RC0603FR-07100KL:RC0603FR-07100KL
Connections:
- net +3.3V: now also R21.1
- net +5V: now also J6.4 (Pin_4)
- net CANH: now also J6.3 (Pin_3)
- net CANL: now also J6.2 (Pin_2)
- net CAN_TERM: now also R21.2
- net GND: now also J3.1 (Pin_1), J6.1 (Pin_1)
- net PA15: now also J3.3 (Pin_3)
- net PA19: now also J3.2 (Pin_2)
- net VAA: now also J3.4 (Pin_4)

Commit message: Use BeagleConnect product names consistently
Other:
- title: AM13E QuadESC SoM — IO connectors -> BeagleConnect Torque — IO connectors
Changed lines of the file:
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@@
 	(paper "USLetter")
 	(title_block
-		(title "AM13E QuadESC SoM — IO connectors")
+		(title "BeagleConnect Torque — IO connectors")
 		(date "2026-08-06")
 		(rev "A")
