File: som/mcu-core.kicad_sch (KiCad schematic)
At the start: 31 parts, among them U1 XAM13E23019GTPZ, Y1 ECS-250-12-33-AGN-TR

Commit message: Initial layout completed
Parts:
- removed D1: LED, LED_SMD:LED_0402_1005Metric, symbol Device:LED
- removed R10, R6: 10k, Resistor_SMD:R_0201_0603Metric, symbol RC0603FR-07100KL:RC0603FR-07100KL
- removed R11, R12: 4.7k, Resistor_SMD:R_0201_0603Metric, symbol RC0603FR-07100KL:RC0603FR-07100KL
- removed R3, R4: 0, Resistor_SMD:R_0201_0603Metric, symbol Device:R
- removed R8: 2.2k, Resistor_SMD:R_0201_0603Metric, symbol RC0603FR-07100KL:RC0603FR-07100KL
- removed R9: 1.5k, Resistor_SMD:R_0201_0603Metric, symbol RC0603FR-07100KL:RC0603FR-07100KL
- renumbered C23 to C12, C12 to C13, C13 to C14, R7 to R6, R13 to R7
Connections:
- net GNDA is gone; now on net GND: C2.2, C4.1, C6.1, U1.23 (VSSA)
- net GNDREF is gone; now on net GND: C10.2, C11.1, C12.1, U1.35 (VREFLO)
- net PB3: now reaches U1.18 (PB3_AIN5)
- net PB6: now reaches U1.65 (PB6)
- net PB9: now reaches U1.68 (PB9)
- net PB12: now reaches U1.81 (PB12)
- net PB18: now reaches U1.84 (PB18)
- net PB19: now reaches U1.85 (PB19)
- net PB20: now reaches U1.86 (PB20)
- net PB21: now reaches U1.87 (PB21)
- net PB22: now reaches U1.88 (PB22)
- net PB23: now reaches U1.89 (PB23)
- net PC18: now reaches U1.19 (PC18)
- net PC0: now reaches U1.97 (PC0)
- net PA4: now reaches U1.26 (PA4_AIN10)
- net PA5: now reaches U1.27 (PA5_AIN11)
- net PA12: now reaches U1.73 (PA12)
- net PA20: now reaches U1.91 (PA20)
- net PA22: now reaches U1.93 (PA22)
- net PA23: now reaches U1.94 (PA23)
- net PA25: now reaches U1.96 (PA25)
- net BSL_INVOKE renamed PB16
- net CAN_RX renamed PA21
- net CAN_TX renamed PA8
- net DRV_ENABLE renamed PA17
- net DSHOT1 renamed PA18
- net DSHOT2 renamed PA15
- net DSHOT3 renamed PB10
- net DSHOT4 renamed PB11
- net M1_BEMFA renamed PA0
- net M1_BEMFB renamed PA1
- net M1_BEMFC renamed PA2
- net M1_IA renamed PC10
- net M1_IB renamed PC11
- net M1_IC renamed PC12
- net M1_PWMA renamed PA11
- net M1_PWMC renamed PA10
- net M2_BEMFA renamed PB0
- net M2_BEMFB renamed PB1
- net M2_BEMFC renamed PB2
- net M2_IA renamed PC13
- net M2_IB renamed PC14
- net M2_IC renamed PC15
- net M2_PWMA renamed PB17
- net M2_PWMB renamed PB7
- net M2_PWMC renamed PB8
- net M3_BEMFA renamed PC9
- net M3_BEMFB renamed PC7
- net M3_BEMFC renamed PC8
- net M3_IA renamed PA30
- net M3_IB renamed PA31
- net M3_IC renamed PB24
- net M3_PWMA renamed PC1
- net M3_PWMB renamed PB28
- net M3_PWMC renamed PA24
- net M4_BEMFA renamed PA27
- net M4_BEMFB renamed PA28
- net M4_BEMFC renamed PA29
- net M4_IA renamed PB25
- net M4_IB renamed PB26
- net M4_IC renamed PB27
- net M4_PWMA renamed PA6
- net M4_PWMB renamed PA3
- net PA3: no longer U1.70 (PA9_AIN43)
- net M4_PWMC renamed PA7
- net M_TEMP1 renamed PB29
- net M_TEMP2 renamed PB30
- net M_TEMP3 renamed PB31
- net M_TEMP4 renamed PB5
- net NRST renamed nRST
- net SPI_MISO renamed PC3
- net SPI_MOSI renamed PC6
- net SPI_SCLK renamed PC2
- net SPI_nCS0 renamed PC4
- net SPI_nCS1 renamed PC5
- net SPI_nCS3 renamed PB13
- net SPI_nCS4 renamed PB14
- net STATUS_LED renamed PB4
- net SWCLK renamed PA14
- net SWDIO renamed PA13
- net SWO renamed PA19
- net VBAT_SNS renamed PA26
- net VREF_IN renamed VAA
- net nFAULT2 renamed PB15
- net PB15: no longer U1.10 (PC25)
- net nFAULT3 renamed PC26
- net nFAULT4 renamed PA16
- new net PA9: U1.70 (PA9_AIN43)
- new net PC25: U1.10 (PC25)

Commit message: Use BeagleConnect product names consistently
Other:
- title: AM13E QuadESC SoM — MCU core -> BeagleConnect Torque — MCU core
Changed lines of the file:
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@@
 	(paper "USLetter")
 	(title_block
-		(title "AM13E QuadESC SoM — MCU core")
+		(title "BeagleConnect Torque — MCU core")
 		(date "2026-08-06")
 		(rev "A")
