File: som/power.kicad_sch (KiCad schematic)
At the start: 11 parts, among them U3 TPS2116DRLR, U4 TPS22950YBHR, U5 TPS7A2633DRVR

Commit message: Initial layout completed
Parts:
- renumbered R20 to R18, R21 to R19, R22 to R20, U3 to U4, U4 to U5, U5 to U6
Changed lines of the file:
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@@
 		(dnp no)
 		(fields_autoplaced yes)
-		(property "Reference" "#PWR035"
+		(property "Reference" "#PWR046"
 			(at 161.29 165.1 0)
 			(hide yes)
@@
 			(project "som"
 				(path "/e4559485-d7d4-484b-a95c-f1b86ccdac46/42e4fcf3-735d-4282-a598-f4243dbc0439"
-					(reference "#PWR035")
+					(reference "#PWR046")
 					(unit 1)
 				)
@@
 		(dnp no)
 		(fields_autoplaced yes)
-		(property "Reference" "#PWR028"
+		(property "Reference" "#PWR039"
 			(at 90.17 101.6 0)
 			(hide yes)
@@
 			(project "som"
 				(path "/e4559485-d7d4-484b-a95c-f1b86ccdac46/42e4fcf3-735d-4282-a598-f4243dbc0439"
-					(reference "#PWR028")
+					(reference "#PWR039")
 					(unit 1)
 				)
@@
 		(dnp no)
 		(fields_autoplaced yes)
-		(property "Reference" "U5"
+		(property "Reference" "U6"
 			(at 121.92 74.93 0)
 			(show_name no)
@@
 			(project "som"
 				(path "/e4559485-d7d4-484b-a95c-f1b86ccdac46/42e4fcf3-735d-4282-a598-f4243dbc0439"
-					(reference "U5")
+					(reference "U6")
 					(unit 1)
 				)
@@
 		(dnp no)
 		(fields_autoplaced yes)
-		(property "Reference" "#PWR034"
+		(property "Reference" "#PWR045"
 			(at 152.4 116.84 0)
 			(hide yes)
@@
 			(project "som"
 				(path "/e4559485-d7d4-484b-a95c-f1b86ccdac46/42e4fcf3-735d-4282-a598-f4243dbc0439"
-					(reference "#PWR034")
+					(reference "#PWR045")
 					(unit 1)
 				)
@@
 		(dnp no)
 		(fields_autoplaced yes)
-		(property "Reference" "R22"
+		(property "Reference" "R20"
 			(at 107.95 161.2899 0)
 			(show_name no)
@@
 			(project "som"
 				(path "/e4559485-d7d4-484b-a95c-f1b86ccdac46/42e4fcf3-735d-4282-a598-f4243dbc0439"
-					(reference "R22")
+					(reference "R20")
 					(unit 1)
 				)
@@
 		(dnp no)
 		(fields_autoplaced yes)
-		(property "Reference" "U3"
+		(property "Reference" "U4"
 			(at 139.7 134.62 0)
 			(show_name no)
@@
 			(project "som"
 				(path "/e4559485-d7d4-484b-a95c-f1b86ccdac46/42e4fcf3-735d-4282-a598-f4243dbc0439"
-					(reference "U3")
+					(reference "U4")
 					(unit 1)
 				)
@@
 		(dnp no)
 		(fields_autoplaced yes)
-		(property "Reference" "#PWR027"
+		(property "Reference" "#PWR038"
 			(at 83.82 88.9 0)
 			(hide yes)
@@
 			(project "som"
 				(path "/e4559485-d7d4-484b-a95c-f1b86ccdac46/42e4fcf3-735d-4282-a598-f4243dbc0439"
-					(reference "#PWR027")
+					(reference "#PWR038")
 					(unit 1)
 				)
@@
 		(dnp no)
 		(fields_autoplaced yes)
-		(property "Reference" "U4"
+		(property "Reference" "U5"
 			(at 121.92 31.75 0)
 			(show_name no)
@@
 			(project "som"
 				(path "/e4559485-d7d4-484b-a95c-f1b86ccdac46/42e4fcf3-735d-4282-a598-f4243dbc0439"
-					(reference "U4")
+					(reference "U5")
 					(unit 1)
 				)
@@
 		(dnp no)
 		(fields_autoplaced yes)
-		(property "Reference" "R21"
+		(property "Reference" "R19"
 			(at 107.95 152.3999 0)
 			(show_name no)
@@
 			(project "som"
 				(path "/e4559485-d7d4-484b-a95c-f1b86ccdac46/42e4fcf3-735d-4282-a598-f4243dbc0439"
-					(reference "R21")
+					(reference "R19")
 					(unit 1)
 				)
@@
 		(dnp no)
 		(fields_autoplaced yes)
-		(property "Reference" "#PWR036"
+		(property "Reference" "#PWR047"
 			(at 173.99 148.59 0)
 			(hide yes)
@@
 			(project "som"
 				(path "/e4559485-d7d4-484b-a95c-f1b86ccdac46/42e4fcf3-735d-4282-a598-f4243dbc0439"
-					(reference "#PWR036")
+					(reference "#PWR047")
 					(unit 1)
 				)
@@
 		(dnp no)
 		(fields_autoplaced yes)
-		(property "Reference" "#PWR030"
+		(property "Reference" "#PWR041"
 			(at 101.6 66.04 0)
 			(hide yes)
@@
 			(project "som"
 				(path "/e4559485-d7d4-484b-a95c-f1b86ccdac46/42e4fcf3-735d-4282-a598-f4243dbc0439"
-					(reference "#PWR030")
+					(reference "#PWR041")
 					(unit 1)
 				)
@@
 		(dnp no)
 		(fields_autoplaced yes)
-		(property "Reference" "#PWR033"
+		(property "Reference" "#PWR044"
 			(at 151.13 43.18 0)
 			(hide yes)
@@
 			(project "som"
 				(path "/e4559485-d7d4-484b-a95c-f1b86ccdac46/42e4fcf3-735d-4282-a598-f4243dbc0439"
-					(reference "#PWR033")
+					(reference "#PWR044")
 					(unit 1)
 				)
@@
 		(dnp no)
 		(fields_autoplaced yes)
-		(property "Reference" "#PWR029"
+		(property "Reference" "#PWR040"
 			(at 93.98 41.91 0)
 			(hide yes)
@@
 			(project "som"
 				(path "/e4559485-d7d4-484b-a95c-f1b86ccdac46/42e4fcf3-735d-4282-a598-f4243dbc0439"
-					(reference "#PWR029")
+					(reference "#PWR040")
 					(unit 1)
 				)
@@
 		(dnp no)
 		(fields_autoplaced yes)
-		(property "Reference" "#PWR031"
+		(property "Reference" "#PWR042"
 			(at 105.41 173.99 0)
 			(hide yes)
@@
 			(project "som"
 				(path "/e4559485-d7d4-484b-a95c-f1b86ccdac46/42e4fcf3-735d-4282-a598-f4243dbc0439"
-					(reference "#PWR031")
+					(reference "#PWR042")
 					(unit 1)
 				)
@@
 		(dnp no)
 		(fields_autoplaced yes)
-		(property "Reference" "R20"
+		(property "Reference" "R18"
 			(at 104.14 52.0699 0)
 			(show_name no)
@@
 			(project "som"
 				(path "/e4559485-d7d4-484b-a95c-f1b86ccdac46/42e4fcf3-735d-4282-a598-f4243dbc0439"
-					(reference "R20")
+					(reference "R18")
 					(unit 1)
 				)
@@
 		(dnp no)
 		(fields_autoplaced yes)
-		(property "Reference" "#PWR032"
+		(property "Reference" "#PWR043"
 			(at 144.78 59.69 0)
 			(hide yes)
@@
 			(project "som"
 				(path "/e4559485-d7d4-484b-a95c-f1b86ccdac46/42e4fcf3-735d-4282-a598-f4243dbc0439"
-					(reference "#PWR032")
-					(unit 1)
-				)
+					(reference "#PWR043")
+					(unit 1)
+				)

Commit message: Use BeagleConnect product names consistently
Other:
- title: AM13E QuadESC SoM — Power -> BeagleConnect Torque — Power
Changed lines of the file:
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@@
 	(paper "USLetter")
 	(title_block
-		(title "AM13E QuadESC SoM — Power")
+		(title "BeagleConnect Torque — Power")
 		(date "2026-08-06")
 		(rev "A")
