File: som/som.kicad_sch (KiCad schematic)
At the start: 0 parts

Commit message: Use BeagleConnect product names consistently
Other:
- title: AM13E QuadESC SoM — Root / block diagram -> BeagleConnect Torque — Root / block diagram
Changed lines of the file:
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@@
 	(paper "USLetter")
 	(title_block
-		(title "AM13E QuadESC SoM — Root / block diagram")
+		(title "BeagleConnect Torque — Root / block diagram")
 		(date "2026-08-06")
 		(rev "A")
